File: Lab03/Lab03Schmatics/Lab03Schmatics.sch (KiCad schematic (older format))
At the start: 9 parts, among them J1 Arduino_Mega_Header, U2 osoyoo_voltage_display

Commit message: updated schematic for lab 3 part 2
Parts:
- added U?: kettering_light_sensor, symbol custom:kettering_light_sensor
Connections:
- net at J1.17 (AD8): now also U?.~ (S3)
- net at J1.18 (AD9): now also U?.~ (S3)
- net at J1.19 (AD10): now also U?.~ (S3)
- net at right.~ (VD): now also BT?.2 (-)
- net at left.~ (VD): no longer right.~ (VD)
- new net: left.~ (VD), right.~ (VD) (x2)
- new net: U2.~ (Vt), right.~ (VD) (x2)
- new net: U?.~ (VCC), U?.~ (VCC)
- now unconnected: left.~ (VD)
Changed lines of the file:
@@
 Wire Wire Line
 	4800 2200 4700 2200
+$Comp
+L custom:kettering_light_sensor U?
+U 1 1 5E468391
+P 2100 3000
+F 0 "U?" H 2167 2035 50  0000 C CNN
+F 1 "kettering_light_sensor" H 2167 2126 50  0000 C CNN
+F 2 "" H 2100 3000 50  0001 C CNN
+F 3 "" H 2100 3000 50  0001 C CNN
+	1    2100 3000
+	-1   0    0    1
+$EndComp
+Wire Wire Line
+	3650 3900 3400 3900
+Wire Wire Line
+	3400 3900 3400 2550
+Wire Wire Line
+	3400 2550 2200 2550
+Wire Wire Line
+	3700 3850 3450 3850
+Wire Wire Line
+	3450 2400 2200 2400
+Wire Wire Line
+	3450 2400 3450 3850
+Wire Wire Line
+	2200 2250 3500 2250
+Wire Wire Line
+	3500 2250 3500 3800
+Wire Wire Line
+	3500 3800 3650 3800
 $EndSCHEMATC
